File: esp32vga-keypad/esp32vga-keypad.kicad_pcb (KiCad board)
At the start: 2 copper layers, 81 x 36 mm, 14 parts, among them J1 KEYPAD, SW1 LEFT, SW2 UP, SW3 RIGHT, SW4 DOWN, SW5 RST

Commit message: Update to rev3
Parts:
- J1: footprint Connector_IDC:IDC-Header_2x05_P2.54mm_Vertical -> Connector_IDC:IDC-Header_2x05_P2.54mm_Horizontal
- R1: moved to F.Cu
- SW1, SW2, SW3, SW4, SW5: footprint Button_Switch_SMD:SW_Push_1P1T_NO_6x6mm_H9.5mm -> ESP32S3-VGA-KEYPAD:SW_Push_TS04_NO_6x6mm_H5.00_BKXXX_SMT
- moved R1 61.9 mm to (134.5, 114.9), turned to 180 degrees
- moved SW5 1.47 mm to (145.5, 97.1)
Connections:
- H1 pad 1: (no net) -> GND
- H2 pad 1: (no net) -> GND
- H3 pad 1: (no net) -> GND
- H4 pad 1: (no net) -> GND
Routing:
- net +3.3V: track 9.45 -> 68.4 mm
- net Net-(D1-A): track 66.5 -> 9.52 mm, vias 1 -> 0
- net /K_UP: track 28.9 -> 38.2 mm
- net /RST: track 63.9 -> 71.8 mm
- net /K_DOWN: track 44.2 -> 45.0 mm
Other:
- board text added: "ESP32S3-RT-VGA KEYPAD (c)2024 Mario Goegel rev 2"
- board text added: "JLCJLCJLCJLC"
