File: esp32vga-keypad/esp32vga-keypad.kicad_sch (KiCad schematic)
At the start: 14 parts, among them J1 KEYPAD, SW1 LEFT, SW2 UP, SW3 RIGHT, SW4 DOWN, SW5 RST

Commit message: Update to rev3
Parts:
- H1, H2, H3, H4: symbol Mechanical:MountingHole -> Mechanical:MountingHole_Pad
- J1: footprint Connector_IDC:IDC-Header_2x05_P2.54mm_Vertical -> Connector_IDC:IDC-Header_2x05_P2.54mm_Horizontal
- SW1, SW2, SW3, SW4, SW5: footprint Button_Switch_SMD:SW_Push_1P1T_NO_6x6mm_H9.5mm -> ESP32S3-VGA-KEYPAD:SW_Push_TS04_NO_6x6mm_H5.00_BKXXX_SMT
Connections:
- net GND: now also H1.1, H2.1, H3.1, H4.1
Other:
- company: (none) -> Mario Goegel
- title: (none) -> ESP32S3 ROBOTRON VGA ADAPTER - KEYPAD
