File: pc1715-esp32vga/pc1715-esp32vga.kicad_pcb (KiCad board)
At the start: 2 copper layers, 112 x 45 mm, 31 parts, among them J1 IDC10_VIDEO_IN, J2 VGAOUT, J3 USB_B, J4 KEYPAD, J5 IDC16_VGAOUT, J6 USB_C_Receptacle_USB2.0_16P, J7 DBG, U1 LM1117MP-3.3, U2 ESP32-S3-WROOM-1

Commit message: Silkscreen correction for J4 Changed BOOT jumper to PROG jumper, Connection to GND instead VCC
Parts:
- JP1: value BOOT -> PROG
Connections:
- JP1 pad 2: +3.3V -> GND
Routing:
- net +3.3V: track 157.0 -> 115.6 mm
Other:
- board text added: "Robotron VGA Adapter Design (c)2024 M. Goegel Rev 3"
- board text added: "→ ← SY x G ↓ ↑ ST RST 3.3"
- board text removed: "Robotron VGA Adapter Design (c)2024 M. Goegel Rev 2"
- board text removed: "→ ← ST 3.3 G ↓ ↑ SY RST"
Changed lines of the file:
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@@
 			)
 		)
-		(property "Description" ""
+		(property "Description" "ESP32S3WRM1N8R8"
 			(at 0 0 0)
 			(unlocked yes)
@@
 			)
 		)
-		(property "Value" "BOOT"
+		(property "Value" "PROG"
 			(at 0 4.87 90)
 			(layer "F.SilkS")
@@
 			(layers "*.Cu" "*.Mask")
 			(remove_unused_layers no)
-			(net 6 "+3.3V")
+			(net 5 "GND")
 			(pinfunction "B")
 			(pintype "passive")
@@
 		)
 	)
-	(gr_text "Robotron VGA Adapter\nDesign (c)2024 M. Goegel\nRev 2"
+	(gr_text "Robotron VGA Adapter\nDesign (c)2024 M. Goegel\nRev 3"
 		(at 75.3 126.1 0)
 		(layer "F.SilkS")
@@
 		)
 	)
-	(gr_text "→ ← ST 3.3 G\n↓ ↑ SY RST\n\n\n"
-		(at 134.2 132.9 0)
+	(gr_text "→ ←  SY   x   G\n↓ ↑  ST  RST 3.3\n\n\n"
+		(at 133.9 132.95 0)
 		(layer "F.SilkS")
 		(effects
@@
 	)
 	(segment
-		(start 144.9 102.816)
-		(end 167.306129 102.816)
-		(width 0.25)
-		(layer "B.Cu")
-		(net 6)
-	)
-	(segment
 		(start 111.956 122.898)
 		(end 109.0375 125.8165)
@@
 	)
 	(segment
-		(start 167.306129 102.816)
-		(end 169.175 104.684871)
-		(width 0.25)
-		(layer "B.Cu")
-		(net 6)
-	)
-	(segment
 		(start 125.6505 106.2915)
 		(end 125.6505 110.5915)
@@
 	)
 	(segment
-		(start 169.175 104.684871)
-		(end 169.175 118.49)
-		(width 0.25)
-		(layer "B.Cu")
-		(net 6)
-	)
-	(segment
 		(start 126.942 122.158)
 		(end 126.942 113.484)
@@
 		(layer "B.Cu")
 		(net 6)
-	)
-	(segment
-		(start 169.175 118.49)
-		(end 167.365 120.3)
-		(width 0.25)
-		(layer "B.Cu")
-		(net 6)

Commit message: Update to rev3
Parts:
- removed D2: POWER, Diode_SMD:D_0805_2012Metric_Pad1.15x1.40mm_HandSolder
- added D4: SD103BW, Diode_SMD:D_SOD-123, F.Cu at (120.4, 124.5)
- added D5: SD103BW, Diode_SMD:D_SOD-123, F.Cu at (120.4, 126.8)
- added D6: SD103BW, Diode_SMD:D_SOD-123, F.Cu at (120.4, 129.1)
- added J8: EXT-5V, Connector_PinHeader_2.54mm:PinHeader_1x02_P2.54mm_Vertical, F.Cu at (67.1, 112.0)
- added JP2: Jumper_3_Open, Jumper:SolderJumper-3_P1.3mm_Open_RoundedPad1.0x1.5mm_NumberLabels, B.Cu at (118.2, 115.2)
- added JP3: USB-VIN, Connector_PinHeader_2.54mm:PinHeader_1x03_P2.54mm_Vertical, F.Cu at (114.3, 119.1)
- D1: value BAT54C Uf 0,24V -> POWER; footprint Package_TO_SOT_SMD:SOT-23 -> Diode_SMD:D_0805_2012Metric_Pad1.15x1.40mm_HandSolder; moved to F.Cu
- R1, R10, R11, R12, R13, R2, R3, R4, R5, R6, R7, R8, R9, U1: moved to F.Cu
- moved R5 50.6 mm to (97.7, 124.5), turned to 180 degrees
- moved R7 50.4 mm to (97.7, 126.5), turned to 180 degrees
- moved R9 50.3 mm to (97.7, 128.4), turned to 180 degrees
- moved R6 46.5 mm to (92.0, 124.5), turned to 0 degrees
- moved R8 46.3 mm to (92.0, 126.5), turned to 0 degrees
- moved R10 46.2 mm to (92.0, 128.4), turned to 0 degrees
- moved D1 26.6 mm to (132.1, 110.7), turned to 90 degrees
- moved R3 15.0 mm to (155.3, 136.2)
- moved R11 13.3 mm to (125.3, 124.5), turned to 180 degrees
- moved R1 12.9 mm to (132.1, 103.6), turned to 90 degrees
- moved R4 12.8 mm to (152.7, 136.2)
- moved R12 11.6 mm to (125.3, 126.8), turned to 180 degrees
- moved R13 10.4 mm to (125.3, 129.1), turned to 180 degrees
- moved C1 5.77 mm to (127.5, 104.1)
- moved C2 5.77 mm to (124.0, 104.1)
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Connections:
- D1 pad 1: /5V_VID -> Net-(D1-K)
- D1 pad 2: /VBUS -> +3.3V
- H1001 pad 1: (no net) -> GND
- H1002 pad 1: (no net) -> GND
- H1003 pad 1: (no net) -> GND
- H1004 pad 1: (no net) -> GND
- J1 pad 10: /BSYNC -> Net-(D6-K)
- J1 pad 4: /VIDEO -> Net-(D4-K)
- J1 pad 6: /INTENS -> Net-(D5-K)
- R2 pad 2: Net-(D2-K) -> Net-(D1-K)
Routing:
- net /R2: track 4.66 -> 80.8 mm, vias 1 -> 4
- net /R1: track 3.87 -> 71.6 mm, vias 1 -> 4
- net /B2: track 4.29 -> 70.8 mm, vias 1 -> 4
- net /G2: track 4.32 -> 67.5 mm, vias 1 -> 2
- net +5V: track 24.6 -> 87.1 mm, vias 1 -> 0
- net /G1: track 4.23 -> 61.2 mm, vias 1 -> 4
- net /B1: track 4.23 -> 61.2 mm, vias 1 -> 4
- net /VSYNC: track 92.0 -> 144.0 mm
- net /HSYNC: track 94.6 -> 143.1 mm
- net /RED: track 106.7 -> 60.1 mm, vias 2 -> 0
- net /GREEN: track 100.1 -> 54.4 mm, vias 2 -> 1
- net GND: track 41.3 -> 0.00 mm, vias 41 -> 43
- net /BLUE: track 98.8 -> 64.7 mm, vias 2 -> 1
- net /K_RIGHT: track 41.1 -> 73.3 mm
- net /VIDEO: track 88.0 -> 60.8 mm, vias 2 -> 3
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Other:
- board text added: "5V GND"
- board text added: "5V SRC USB 1-2 VIDEO-IN 2-3"
- board text added: "Robotron VGA Adapter Design (c)2025 M. Goegel Rev 3"
- board text removed: "Robotron VGA Adapter Design (c)2024 M. Goegel Rev 3"
